File: battery_interface_board.kicad_pcb (KiCad board)
At the start: 6 copper layers, 0 parts

Commit message: PCB[Layout and Routing]: Routing and layout done, changed to micofit connector, need to review and fix drc errors. SCH[Connector & Fuse]: Schmatic for connector, fuse and board to board layout, need to cleanup and add board standoffs.
Parts:
- added F1: 500 mA 125 V, remote_0451.500mrl:0451Series_LTF, F.Cu at (90.5, 159.5)
- added F10: 500 mA 125 V, remote_0451.500mrl:0451Series_LTF, F.Cu at (89.5, 130.5)
- added F11: 500 mA 125 V, remote_0451.500mrl:0451Series_LTF, F.Cu at (90.5, 135.5)
- added F2: 500 mA 125 V, remote_0451.500mrl:0451Series_LTF, F.Cu at (89.5, 164.8)
- added F3: 500 mA 125 V, remote_0451.500mrl:0451Series_LTF, F.Cu at (166.5, 159.5)
- added F4: 500 mA 125 V, remote_0451.500mrl:0451Series_LTF, F.Cu at (221.5, 159.5)
- added F5: 500 mA 125 V, remote_0451.500mrl:0451Series_LTF, F.Cu at (297.5, 159.5)
- added F6: 500 mA 125 V, remote_0451.500mrl:0451Series_LTF, F.Cu at (348.5, 159.5)
- added F7: 500 mA 125 V, remote_0451.500mrl:0451Series_LTF, F.Cu at (297.5, 135.5)
- added F8: 500 mA 125 V, remote_0451.500mrl:0451Series_LTF, F.Cu at (221.5, 135.5)
- added F9: 500 mA 125 V, remote_0451.500mrl:0451Series_LTF, F.Cu at (166.5, 135.5)
- added J1: Step Bushing, remote_n_a:steped_bushing, F.Cu at (80.0, 159.5)
- added J10: IPT1-110-01-L-D, remote_ipt1-110-01-l-d:SAMTEC_IPT1-110-01-L-D, F.Cu at (195.5, 147.5)
- added J11: 0430450409, remote_0430450409:CONN_SD-43045-004_04_MOL, F.Cu at (86.0, 147.5)
- added J12: 0430450409, remote_0430450409:CONN_SD-43045-004_04_MOL, F.Cu at (162.0, 147.5)
- added J13: 0430450409, remote_0430450409:CONN_SD-43045-004_04_MOL, F.Cu at (238.0, 147.5)
- added J14: 0430450409, remote_0430450409:CONN_SD-43045-004_04_MOL, F.Cu at (314.0, 147.5)
- added J2: Step Bushing, remote_n_a:steped_bushing, F.Cu at (156.0, 159.5)
- added J3: Step Bushing, remote_n_a:steped_bushing, F.Cu at (232.0, 159.5)
- added J4: Step Bushing, remote_n_a:steped_bushing, F.Cu at (308.0, 159.5)
- added J5: Step Bushing, remote_n_a:steped_bushing, F.Cu at (359.1, 159.5)
- added J6: Step Bushing, remote_n_a:steped_bushing, F.Cu at (308.0, 135.5)
- added J7: Step Bushing, remote_n_a:steped_bushing, F.Cu at (232.0, 135.5)
- added J8: Step Bushing, remote_n_a:steped_bushing, F.Cu at (156.0, 135.5)
- added J9: Step Bushing, remote_n_a:steped_bushing, F.Cu at (80.0, 135.5)
Routing:
- net /Project Architecture/Connectors/TAP4: track 0.00 -> 155.9 mm
- net /Project Architecture/Connectors/T_P4: track 0.00 -> 118.0 mm, vias 0 -> 1
- net /Project Architecture/Connectors/T_P5: track 0.00 -> 117.8 mm, vias 0 -> 1
- net /Project Architecture/Connectors/T_P8: track 0.00 -> 117.7 mm, vias 0 -> 1
- net /Project Architecture/Connectors/T_P1: track 0.00 -> 117.6 mm, vias 0 -> 1
- net /Project Architecture/Connectors/TAP0: track 0.00 -> 115.5 mm
- net /Project Architecture/Connectors/GND: track 0.00 -> 112.0 mm
- net /Project Architecture/Connectors/TAP8: track 0.00 -> 111.9 mm
- net /Project Architecture/Connectors/VMODULE: track 0.00 -> 110.8 mm
- net /Project Architecture/Connectors/TAP3: track 0.00 -> 102.7 mm
- net /Project Architecture/Connectors/TAP5: track 0.00 -> 102.1 mm
- net /Project Architecture/Connectors/T_P3: track 0.00 -> 45.3 mm, vias 0 -> 1
- net /Project Architecture/Connectors/T_P6: track 0.00 -> 41.8 mm, vias 0 -> 1
- net /Project Architecture/Connectors/T_P7: track 0.00 -> 40.6 mm, vias 0 -> 1
- net /Project Architecture/Connectors/T_P2: track 0.00 -> 40.5 mm
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Other:
- board outline added: 300 x 47 mm
- copper layers 6 -> 4

Commit message: PCB[Routing, Layout]: Need to finish routing ground for temp, and ensure its fine to combine on bms board or route to correct ground plane. Layout mostly done need to check interface in module cad.
Connections:
- J10 pad 04: /Project Architecture/Connectors/T_P8 -> /Project Architecture/Connectors/T_P1
- J10 pad 06: /Project Architecture/Connectors/T_P7 -> /Project Architecture/Connectors/T_P2
- J10 pad 08: /Project Architecture/Connectors/T_P6 -> /Project Architecture/Connectors/T_P3
- J10 pad 10: /Project Architecture/Connectors/T_P5 -> /Project Architecture/Connectors/T_P4
- J10 pad 12: /Project Architecture/Connectors/T_P4 -> /Project Architecture/Connectors/T_P5
- J10 pad 14: /Project Architecture/Connectors/T_P3 -> /Project Architecture/Connectors/T_P6
- J10 pad 16: /Project Architecture/Connectors/T_P2 -> /Project Architecture/Connectors/T_P7
- J10 pad 18: /Project Architecture/Connectors/T_P1 -> /Project Architecture/Connectors/T_P8
Routing:
- net /Project Architecture/Connectors/T_P3: track 45.3 -> 42.6 mm, vias 1 -> 0
- net /Project Architecture/Connectors/T_P6: track 41.8 -> 39.6 mm, vias 1 -> 0
- net /Project Architecture/Connectors/T_P4: track 118.0 -> 116.5 mm
- net /Project Architecture/Connectors/T_P5: track 117.8 -> 116.3 mm
- net /Project Architecture/Connectors/T_P8: track 117.7 -> 116.4 mm, vias 1 -> 0
- net /Project Architecture/Connectors/T_P7: track 40.6 -> 39.3 mm, vias 1 -> 0
- net /Project Architecture/Connectors/T_P2: track 40.5 -> 39.4 mm
- net /Project Architecture/Connectors/T_P1: track 117.6 -> 116.4 mm, vias 1 -> 0

Commit message: PCB[Mounting]: Added standoffs going to test clearnaces. SCH[Mechanical]: Added standoffs, 14mm metal smt, small naming changes to match bms_slave sch.
Parts:
- added G1: BMD Logo, remote_bmd_logo:BDM_Logo_20mm, F.Cu at (188.3, 220.6)
- added G2: SAE Electric logo, remote_sae_electric_logo:SAE_Electric_Logo_10mm, F.Cu at (201.3, 219.8)
- added MP1: 9774140360R, remote_9774140360r:WA-SMSI_9774140360, F.Cu at (195.5, 166.2)
- added MP2: 9774140360R, remote_9774140360r:WA-SMSI_9774140360, F.Cu at (195.5, 128.8)
- added MP3: 9774140360R, remote_9774140360r:WA-SMSI_9774140360, F.Cu at (142.5, 166.2)
- added MP4: 9774140360R, remote_9774140360r:WA-SMSI_9774140360, F.Cu at (142.5, 128.8)
- turned J10 to -90 degrees
Connections:
- J10 pad 01: /Project Architecture/Connectors/GND -> /Project Architecture/Connectors/TAP8
- J10 pad 02: /Project Architecture/Connectors/TEMP_RTN -> /Project Architecture/Connectors/VMODULE
- J10 pad 03: /Project Architecture/Connectors/TAP0 -> /Project Architecture/Connectors/TAP7
- J10 pad 04: /Project Architecture/Connectors/T_P1 -> /Project Architecture/Connectors/TMP8
- J10 pad 05: /Project Architecture/Connectors/TAP1 -> /Project Architecture/Connectors/TAP6
- J10 pad 06: /Project Architecture/Connectors/T_P2 -> /Project Architecture/Connectors/TMP7
- J10 pad 07: /Project Architecture/Connectors/TAP2 -> /Project Architecture/Connectors/TAP5
- J10 pad 08: /Project Architecture/Connectors/T_P3 -> /Project Architecture/Connectors/TMP6
- J10 pad 09: /Project Architecture/Connectors/TAP3 -> /Project Architecture/Connectors/TAP4
- J10 pad 10: /Project Architecture/Connectors/T_P4 -> /Project Architecture/Connectors/TMP5
- J10 pad 11: /Project Architecture/Connectors/TAP4 -> /Project Architecture/Connectors/TAP3
- J10 pad 12: /Project Architecture/Connectors/T_P5 -> /Project Architecture/Connectors/TMP4
- J10 pad 13: /Project Architecture/Connectors/TAP5 -> /Project Architecture/Connectors/TAP2
- J10 pad 14: /Project Architecture/Connectors/T_P6 -> /Project Architecture/Connectors/TMP3
- J10 pad 15: /Project Architecture/Connectors/TAP6 -> /Project Architecture/Connectors/TAP1
- J10 pad 16: /Project Architecture/Connectors/T_P7 -> /Project Architecture/Connectors/TMP2
- J10 pad 17: /Project Architecture/Connectors/TAP7 -> /Project Architecture/Connectors/TAP0
- J10 pad 18: /Project Architecture/Connectors/T_P8 -> /Project Architecture/Connectors/TMP1
- J10 pad 19: /Project Architecture/Connectors/TAP8 -> /Project Architecture/Connectors/GND
- J10 pad 20: /Project Architecture/Connectors/VMODULE -> /Project Architecture/Connectors/TEMP_RTN
Routing:
- net /Project Architecture/Connectors/TAP4: track 155.9 -> 0.00 mm
- net /Project Architecture/Connectors/T_P4: track 116.5 -> 0.00 mm, vias 1 -> 0
- net /Project Architecture/Connectors/T_P1: track 116.4 -> 0.00 mm
- net /Project Architecture/Connectors/T_P8: track 116.4 -> 0.00 mm
- net /Project Architecture/Connectors/T_P5: track 116.3 -> 0.00 mm, vias 1 -> 0
- net /Project Architecture/Connectors/TAP0: track 115.5 -> 0.00 mm
- net /Project Architecture/Connectors/GND: track 112.0 -> 0.00 mm
- net /Project Architecture/Connectors/TAP8: track 111.9 -> 0.00 mm
- net /Project Architecture/Connectors/VMODULE: track 110.8 -> 0.00 mm
- net /Project Architecture/Connectors/TAP3: track 102.7 -> 0.00 mm
- net /Project Architecture/Connectors/TAP5: track 102.1 -> 0.00 mm
- net /Project Architecture/Connectors/T_P3: track 42.6 -> 0.00 mm
- net /Project Architecture/Connectors/T_P6: track 39.6 -> 0.00 mm
- net /Project Architecture/Connectors/TAP1: track 39.4 -> 0.00 mm
- net /Project Architecture/Connectors/T_P2: track 39.4 -> 0.00 mm
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
Commit message: PCB[Routing, Mechanical, Silk]: Inital routing, Finalized mounting points and board to board connector reltive posision, and inital silkscreen. SCH[Labels]: Updated labels to match BMS_Slave board.
Parts:
- G1: footprint remote_bmd_logo:BDM_Logo_20mm -> remote_bmd_logo:BDM_Logo_40mm
- G2: footprint remote_sae_electric_logo:SAE_Electric_Logo_10mm -> remote_sae_electric_logo:SAE_Electric_Logo_20mm
- moved G2 123.9 mm to (100.7, 147.6)
- moved G1 119.4 mm to (282.5, 147.2)
- moved MP3 0.50 mm to (142.0, 166.2)
- moved MP4 0.50 mm to (142.0, 128.8)
- renumbered F2 to F1, F11 to F10, F10 to F11, F1 to F2
Connections:
- F1 pad 2: /Project Architecture/Connectors/TAP0 -> /Project Architecture/Connectors/GND
- F10 pad 2: /Project Architecture/Connectors/VMODULE -> /Project Architecture/Connectors/TAP8
- F11 pad 2: /Project Architecture/Connectors/TAP8 -> /Project Architecture/Connectors/VMODULE
- F2 pad 2: /Project Architecture/Connectors/GND -> /Project Architecture/Connectors/TAP0
- J11 pad 1: /Project Architecture/Connectors/T_P8 -> /Project Architecture/Connectors/TMP8
- J11 pad 2: /Project Architecture/Connectors/T_P1 -> /Project Architecture/Connectors/TMP1
- J12 pad 1: /Project Architecture/Connectors/T_P7 -> /Project Architecture/Connectors/TMP7
- J12 pad 2: /Project Architecture/Connectors/T_P2 -> /Project Architecture/Connectors/TMP2
- J13 pad 1: /Project Architecture/Connectors/T_P6 -> /Project Architecture/Connectors/TMP6
- J13 pad 2: /Project Architecture/Connectors/T_P3 -> /Project Architecture/Connectors/TMP3
- J14 pad 1: /Project Architecture/Connectors/T_P5 -> /Project Architecture/Connectors/TMP5
- J14 pad 2: /Project Architecture/Connectors/T_P4 -> /Project Architecture/Connectors/TMP4
Routing:
- net /Project Architecture/Connectors/TEMP_RTN: track 0.00 -> 241.4 mm, vias 0 -> 25
- net /Project Architecture/Connectors/TAP4: track 0.00 -> 177.7 mm, vias 0 -> 1
- net /Project Architecture/Connectors/TMP8: track 0.00 -> 119.0 mm
- net /Project Architecture/Connectors/TMP1: track 0.00 -> 118.9 mm
- net /Project Architecture/Connectors/TAP0: track 0.00 -> 113.9 mm, vias 0 -> 2
- net /Project Architecture/Connectors/TMP4: track 0.00 -> 113.1 mm, vias 0 -> 1
- net /Project Architecture/Connectors/TMP5: track 0.00 -> 113.0 mm, vias 0 -> 1
- net /Project Architecture/Connectors/VMODULE: track 0.00 -> 112.0 mm, vias 0 -> 2
- net /Project Architecture/Connectors/GND: track 0.00 -> 111.2 mm, vias 0 -> 2
- net /Project Architecture/Connectors/TAP8: track 0.00 -> 110.9 mm, vias 0 -> 2
- net /Project Architecture/Connectors/TAP3: track 0.00 -> 105.9 mm, vias 0 -> 1
- net /Project Architecture/Connectors/TAP5: track 0.00 -> 105.6 mm
- net /Project Architecture/Connectors/TMP7: track 0.00 -> 41.9 mm
- net /Project Architecture/Connectors/TMP2: track 0.00 -> 41.9 mm
- net /Project Architecture/Connectors/TMP6: track 0.00 -> 37.9 mm
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- added copper zone on B.Cu, net /Project Architecture/Connectors/TEMP_RTN
- added copper zone on F.Cu, net /Project Architecture/Connectors/TEMP_RTN
Other:
- copper layers 4 -> 2
- board text added: "${PROJECT_NAME} REVISION: ${REVISION} RELEASE DATE: ${RELEASE_DATE_NUM} DESIGNER: ${DESIGNER}"

Commit message: PCB[Connector, Clearnces]: Testing clearances.
Parts:
- removed J11, J12, J13, J14: 0430450409, remote_0430450409:CONN_SD-43045-004_04_MOL
- removed J5, J6, J7, J8, J9: Step Bushing, remote_n_a:steped_bushing
- added MP10: Enepaq M5 Clamp, remote_enepaq_m5_clamp:Enepaq_M5_Clamp, F.Cu at (308.0, 135.5)
- added MP11: Enepaq M5 Clamp, remote_enepaq_m5_clamp:Enepaq_M5_Clamp, F.Cu at (232.0, 135.5)
- added MP12: Enepaq M5 Clamp, remote_enepaq_m5_clamp:Enepaq_M5_Clamp, F.Cu at (156.0, 135.5)
- added MP13: Enepaq M5 Clamp, remote_enepaq_m5_clamp:Enepaq_M5_Clamp, F.Cu at (80.0, 135.5)
- added MP5: Enepaq M5 Clamp, remote_enepaq_m5_clamp:Enepaq_M5_Clamp, F.Cu at (80.0, 159.5)
- added MP6: Enepaq M5 Clamp, remote_enepaq_m5_clamp:Enepaq_M5_Clamp, F.Cu at (156.0, 159.5)
- added MP7: Enepaq M5 Clamp, remote_enepaq_m5_clamp:Enepaq_M5_Clamp, F.Cu at (232.0, 159.5)
- added MP8: Enepaq M5 Clamp, remote_enepaq_m5_clamp:Enepaq_M5_Clamp, F.Cu at (308.0, 159.5)
- added MP9: Enepaq M5 Clamp, remote_enepaq_m5_clamp:Enepaq_M5_Clamp, F.Cu at (359.1, 159.5)
- J1, J2, J3, J4: value Step Bushing -> 0436500412; footprint remote_n_a:steped_bushing -> remote_0436500412:CONN_SD-43650-005_04_MOL
- moved J2 44.6 mm to (199.0, 147.8), turned to -90 degrees
- moved J1 43.9 mm to (122.2, 147.5), turned to -90 degrees
- moved J3 43.4 mm to (273.8, 147.8), turned to -90 degrees
- moved J4 43.1 mm to (348.0, 143.5), turned to -90 degrees
- moved F9 25.0 mm to (141.5, 135.5), turned to 180 degrees
- moved J10 24.5 mm to (171.0, 147.5)
- moved MP1 24.5 mm to (171.0, 166.2)
- moved MP2 24.5 mm to (171.0, 128.8)
- moved MP3 24.5 mm to (117.5, 166.2)
- moved MP4 24.5 mm to (117.5, 128.8)
- moved F3 24.0 mm to (142.5, 159.5), turned to 180 degrees
- moved F11 11.0 mm to (92.7, 141.0)
- moved F1 10.8 mm to (92.8, 154.5)
- moved F10 9.31 mm to (89.8, 144.8)
- moved F2 9.04 mm to (90.0, 150.5)
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Connections:
- J1 pad 1: /Project Architecture/Connectors/BUSH1 -> /Project Architecture/Connectors/TMP8
- J2 pad 1: /Project Architecture/Connectors/BUSH2 -> /Project Architecture/Connectors/TMP7
- J3 pad 1: /Project Architecture/Connectors/BUSH3 -> /Project Architecture/Connectors/TMP6
- J4 pad 1: /Project Architecture/Connectors/BUSH4 -> /Project Architecture/Connectors/TMP5
Routing:
- net /Project Architecture/Connectors/TEMP_RTN: track 241.4 -> 0.00 mm, vias 25 -> 0
- net /Project Architecture/Connectors/TMP8: track 119.0 -> 0.00 mm
- net /Project Architecture/Connectors/TMP1: track 118.9 -> 0.00 mm
- net /Project Architecture/Connectors/TMP4: track 113.1 -> 0.00 mm, vias 1 -> 0
- net /Project Architecture/Connectors/TMP5: track 113.0 -> 0.00 mm, vias 1 -> 0
- net /Project Architecture/Connectors/TMP7: track 41.9 -> 0.00 mm
- net /Project Architecture/Connectors/TMP2: track 41.9 -> 0.00 mm
- net /Project Architecture/Connectors/TMP6: track 37.9 -> 0.00 mm
- net /Project Architecture/Connectors/TMP3: track 37.9 -> 0.00 mm
- net /Project Architecture/Connectors/TAP8: track 110.9 -> 75.1 mm, vias 2 -> 1
- net /Project Architecture/Connectors/TAP0: track 113.9 -> 81.1 mm, vias 2 -> 1
- net /Project Architecture/Connectors/GND: track 111.2 -> 80.2 mm, vias 2 -> 1
- net /Project Architecture/Connectors/VMODULE: track 112.0 -> 83.5 mm, vias 2 -> 1
- net /Project Architecture/Connectors/TAP6: track 28.1 -> 52.0 mm
- net /Project Architecture/Connectors/TAP2: track 28.2 -> 51.0 mm
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- removed copper zone on B.Cu, net /Project Architecture/Connectors/TEMP_RTN
- removed copper zone on F.Cu, net /Project Architecture/Connectors/TEMP_RTN

Commit message: PCB[Routing, Mount]: Did intial routing and clearnce, Changed connector from Microfit 3.0 to JST XH STM 4 Position. More room and mating end fit fully on board surface. Need to update standoffs, and samtech board to board connctor.
Parts:
- G1: moved to B.Cu
- J1, J2, J3, J4: value 0436500412 -> S4B-XH-SM4-TB; footprint remote_0436500412:CONN_SD-43650-005_04_MOL -> remote_s4b-xh-sm4-tb:JST_S4B-XH-SM4-TB
- moved G2 246.9 mm to (347.0, 131.5)
- moved G1 78.0 mm to (204.5, 146.5), turned to 180 degrees
- moved F6 20.6 mm to (359.1, 147.5)
- moved F5 9.60 mm to (297.5, 150.5)
- moved F7 9.60 mm to (297.5, 144.5)
- moved F4 8.96 mm to (221.0, 151.0)
- moved F8 8.96 mm to (221.0, 144.0)
- moved J2 7.50 mm to (191.5, 147.5)
- moved J1 6.75 mm to (115.5, 147.5)
- moved J3 6.27 mm to (267.5, 147.5)
- moved J4 6.02 mm to (343.5, 147.5)
- moved F9 3.56 mm to (144.0, 138.0), turned to -90 degrees
- moved F3 2.94 mm to (144.0, 157.0), turned to 90 degrees
- moved F2 0.56 mm to (89.8, 150.0)
- moved F1 0.50 mm to (92.8, 154.0)
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Connections:
- J1 pad 2: /Project Architecture/Connectors/TMP1 -> /Project Architecture/Connectors/TEMP_RTN
- J1 pad 4: /Project Architecture/Connectors/TEMP_RTN -> /Project Architecture/Connectors/TMP1
- J2 pad 2: /Project Architecture/Connectors/TMP2 -> /Project Architecture/Connectors/TEMP_RTN
- J2 pad 4: /Project Architecture/Connectors/TEMP_RTN -> /Project Architecture/Connectors/TMP2
- J3 pad 2: /Project Architecture/Connectors/TMP3 -> /Project Architecture/Connectors/TEMP_RTN
- J3 pad 4: /Project Architecture/Connectors/TEMP_RTN -> /Project Architecture/Connectors/TMP3
- J4 pad 2: /Project Architecture/Connectors/TMP4 -> /Project Architecture/Connectors/TEMP_RTN
- J4 pad 4: /Project Architecture/Connectors/TEMP_RTN -> /Project Architecture/Connectors/TMP4
Routing:
- net /Project Architecture/Connectors/TMP4: track 0.00 -> 179.1 mm, vias 0 -> 1
- net /Project Architecture/Connectors/TMP5: track 0.00 -> 179.0 mm, vias 0 -> 1
- net /Project Architecture/Connectors/TMP6: track 0.00 -> 104.5 mm, vias 0 -> 1
- net /Project Architecture/Connectors/TMP3: track 0.00 -> 104.5 mm, vias 0 -> 1
- net /Project Architecture/Connectors/TMP1: track 0.00 -> 57.3 mm
- net /Project Architecture/Connectors/TMP8: track 0.00 -> 55.9 mm
- net /Project Architecture/Connectors/TMP7: track 0.00 -> 27.7 mm
- net /Project Architecture/Connectors/TMP2: track 0.00 -> 27.7 mm
- net /Project Architecture/Connectors/BUSH9: track 0.00 -> 26.1 mm
- net /Project Architecture/Connectors/BUSH1: track 0.00 -> 26.1 mm
- net /Project Architecture/Connectors/BUSH4: track 0.00 -> 13.5 mm
- net /Project Architecture/Connectors/BUSH6: track 0.00 -> 13.4 mm
- net /Project Architecture/Connectors/BUSH3: track 0.00 -> 13.2 mm
- net /Project Architecture/Connectors/BUSH7: track 0.00 -> 13.1 mm
- net /Project Architecture/Connectors/BUSH5: track 0.00 -> 13.1 mm
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- added copper zone on F.Cu, net /Project Architecture/Connectors/TEMP_RTN
